File: Kicad/V0.1/nightUSB/nightUSB.kicad_sch (KiCad schematic)
At the start: 15 parts, among them J1 TC2030-MCP-NL, J2 USB_A_PLUG, J3 M20-9990546, J4 M20-9990546, U1 PIC18F14K50, Y1 12Mhz

Commit message: Update documentation
Other:
- company: (none) -> Making Devices
- title: (none) -> NightUSB
